Commit message: Further model cleanup, standardize link and joint names.

File: mycobot_description/urdf/mycobot_280/mycobot_280.urdf (robot description, URDF)
Before this commit: robot firefighter, 7 links, 6 joints
Links:
- added link dummy

File: mycobot_description/urdf/mycobot_280/mycobot_280_fixed.urdf (robot description, URDF)
Before this commit: robot firefighter, 7 links, 6 joints
Links:
- removed link joint1
- removed link joint2
- removed link joint3
- removed link joint4
- removed link joint5
- removed link joint6
- removed link joint6_flange
- added link base, mass 0.1; collision mesh filename=package://mycobot_description/urdf/mycobot_280/joint1.dae; visual mesh filename=package://mycobot_description/urdf/mycobot_280/joint1.dae
- added link dummy
- added link link1, mass 0.1; collision mesh filename=package://mycobot_description/urdf/mycobot_280/joint2.dae; visual mesh filename=package://mycobot_description/urdf/mycobot_280/joint2.dae
- added link link2, mass 0.1; collision mesh filename=package://mycobot_description/urdf/mycobot_280/joint3.dae; visual mesh filename=package://mycobot_description/urdf/mycobot_280/joint3.dae
- added link link3, mass 0.1; collision mesh filename=package://mycobot_description/urdf/mycobot_280/joint4.dae; visual mesh filename=package://mycobot_description/urdf/mycobot_280/joint4.dae
- added link link4, mass 0.1; collision mesh filename=package://mycobot_description/urdf/mycobot_280/joint5_fixed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; visual mesh filename=package://mycobot_description/urdf/mycobot_280/joint5_fixed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
- added link link5, mass 0.1; collision mesh filename=package://mycobot_description/urdf/mycobot_280/joint6.dae; visual mesh filename=package://mycobot_description/urdf/mycobot_280/joint6.dae
- added link link6, mass 0.1; collision mesh filename=package://mycobot_description/urdf/mycobot_280/joint7.dae; visual mesh filename=package://mycobot_description/urdf/mycobot_280/joint7.dae
Joints:
- removed joint joint2_to_joint1
- removed joint joint3_to_joint2
- removed joint joint4_to_joint3
- removed joint joint5_to_joint4
- removed joint joint6_to_joint5
- removed joint joint6output_to_joint6
- added joint dummy_joint: type fixed, parent dummy, child base
- added joint link1_to_base: type revolute, parent base, child link1, origin xyz=0 0 0.13156 rpy=0 0 0, axis 0 0 1, limit lower=-3.14 upper=3.14159 effort=1000.0 velocity=0
- added joint link2_to_link1: type revolute, parent link1, child link2, origin xyz=0 0  0 rpy=0 1.5708 -1.5708, axis 0 0 1, limit lower=-3.14 upper=3.14159 effort=1000.0 velocity=0
- added joint link3_to_link2: type revolute, parent link2, child link3, origin xyz=  -0.1104 0 0  rpy=0 0 0, axis 0 0 1, limit lower=-3.14 upper=3.14159 effort=1000.0 velocity=0
- added joint link4_to_link3: type revolute, parent link3, child link4, origin xyz=-0.096 0 0.06462 rpy=0 0 -1.5708, axis 0 0 1, limit lower=-3.14 upper=3.14159 effort=1000.0 velocity=0
- added joint link5_to_link4: type revolute, parent link4, child link5, origin xyz=0 -0.07318 0 rpy=1.5708 -1.5708 0, axis 0 0 1, limit lower=-3.14 upper=3.14159 effort=1000.0 velocity=0
- added joint link6_to_link5: type revolute, parent link5, child link6, origin xyz=0 0.0456 0 rpy=-1.5708 0 0, axis 0 0 1, limit lower=-3.14 upper=3.14159 effort=1000.0 velocity=0

File: mycobot_description/urdf/mycobot_320/mycobot_320.urdf (robot description, URDF)
Before this commit: robot firefighter, 8 links, 7 joints
Links:
- added link dummy
Joints:
- removed joint gitpper_to_joint6output
- removed joint joint2_to_joint1
- removed joint joint3_to_joint2
- removed joint joint4_to_joint3
- removed joint joint5_to_joint4
- removed joint joint6_to_joint5
- removed joint joint6output_to_joint6
- added joint dummy_joint: type fixed, parent dummy, child base
- added joint gripper_to_link6: type fixed, parent link6, child gripper, origin xyz=0 0 0 rpy=0 0 0, axis 0 0 0, limit lower=-3.14 upper=3.14159 effort=1000.0 velocity=0
- added joint link1_to_base: type revolute, parent base, child link1, origin xyz=0 0 0.17846 rpy=0 0 0, axis 0 0 1, limit lower=-3.14 upper=3.14159 effort=1000.0 velocity=0
- added joint link2_to_link1: type revolute, parent link1, child link2, origin xyz=0 0 0 rpy=0 -1.57080 1.57080, axis 0 0 1, limit lower=-3.14 upper=3.14159 effort=1000.0 velocity=0
- added joint link3_to_link2: type revolute, parent link2, child link3, origin xyz=0.13635 0 0 rpy=0 0 0, axis  0 0 1, limit lower=-3.14 upper=3.14159 effort=1000.0 velocity=0
- added joint link4_to_link3: type revolute, parent link3, child link4, origin xyz=0.1 0  0.090 rpy=0 0 1.57080, axis  0 0 1, limit lower=-3.14 upper=3.14159 effort=1000.0 velocity=0
- added joint link5_to_link4: type revolute, parent link4, child link5, origin xyz=0 -0.08515 0 rpy=1.57080 -1.57080 0, axis 0 0 1, limit lower=-3.14 upper=3.14159 effort=1000.0 velocity=0
- added joint link6_to_link5: type revolute, parent link5, child link6, origin xyz=0 0.06 0 rpy=-1.57080 0 0, axis 0 0 1, limit lower=-3.14 upper=3.14159 effort=1000.0 velocity=0

File: mycobot_description/urdf/mycobot_320/mycobot_320_fixed.urdf (robot description, URDF)
Before this commit: robot firefighter, 8 links, 7 joints
Links:
- added link dummy
Joints:
- added joint dummy_joint: type fixed, parent dummy, child base
- joint link3_to_link2: axis  0 0 1 -> 0 0 1
- joint link4_to_link3: axis  0 0 1 -> 0 0 1
